File: kicad/tutorial.kicad_pcb (KiCad board)
At the start: 2 copper layers, 95.3 x 71.4 mm, 26 parts

Commit message: finalized pcb, added both kbfirmware json files
Other:
- board text added: "Pro Micro here (face down) for LEFT HAND VERSION"
- board text added: "Pro Micro here (face down) for RIGHT HAND VERSION"
- board text removed: "Pro Micro here (face down)"
Changed lines of the file:
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@@
   (general
     (thickness 1.6)
-    (drawings 24)
+    (drawings 25)
     (tracks 152)
     (zones 0)
@@
     (40 Dwgs.User user)
     (41 Cmts.User user)
-    (42 Eco1.User user hide)
+    (42 Eco1.User user)
     (43 Eco2.User user)
     (44 Edge.Cuts user)
@@
     (pad 1 np_thru_hole circle (at 0 0) (size 2.2 2.2) (drill 2.2) (layers *.Cu *.Mask))
   )
+  (gr_text "Pro Micro here (face down)\nfor RIGHT HAND VERSION\n" (at 152.4 39.878 270) (layer F.SilkS)
+    (effects (font (size 1.5 1.2) (thickness 0.15)))
+  )
   (gr_line (start 142.875 21.43125) (end 142.875 16.66875) (layer Edge.Cuts) (width 0.12))
   (gr_line (start 147.6375 21.43125) (end 142.875 21.43125) (layer Edge.Cuts) (width 0.12))
@@
     (effects (font (size 2.7 1.9) (thickness 0.475)) (justify left mirror))
   )
-  (gr_text "Pro Micro here\n(face down)\n" (at 152.4 39.878 270) (layer B.SilkS)
-    (effects (font (size 1.5 1.5) (thickness 0.15)) (justify mirror))
+  (gr_text "Pro Micro here (face down)\nfor LEFT HAND VERSION\n" (at 152.4 39.878 270) (layer B.SilkS)
+    (effects (font (size 1.5 1.2) (thickness 0.15)) (justify mirror))
   )
   (gr_text "Pimentoso hardware 2019" (at 142.494 79.756) (layer B.SilkS)
