File: kicad/tutorial.sch (KiCad schematic (older format))
At the start: 26 parts

Commit message: fix lib broken links
Parts:
- MX0, MX1, MX2, MX3, MX4, MX5, MX6, MX7, MX8, MX9: symbol switch:MX-NoLED -> tutorial-rescue:MX-NoLED-switch
Changed lines of the file:
@@
 NoConn ~ 6150 5800
 $Comp
-L switch:MX-NoLED MX0
+L tutorial-rescue:MX-NoLED-switch MX0
 U 1 1 5D1172EF
 P 9200 5400
@@
 $EndComp
 $Comp
-L switch:MX-NoLED MX1
+L tutorial-rescue:MX-NoLED-switch MX1
 U 1 1 5D118615
 P 9700 5400
@@
 $EndComp
 $Comp
-L switch:MX-NoLED MX2
+L tutorial-rescue:MX-NoLED-switch MX2
 U 1 1 5D1188EE
 P 10200 5400
@@
 $EndComp
 $Comp
-L switch:MX-NoLED MX3
+L tutorial-rescue:MX-NoLED-switch MX3
 U 1 1 5D11A3DC
 P 10700 5400
@@
 $EndComp
 $Comp
-L switch:MX-NoLED MX4
+L tutorial-rescue:MX-NoLED-switch MX4
 U 1 1 5D11A6DD
 P 9200 6400
@@
 $EndComp
 $Comp
-L switch:MX-NoLED MX5
+L tutorial-rescue:MX-NoLED-switch MX5
 U 1 1 5D11ACF4
 P 9700 6400
@@
 $EndComp
 $Comp
-L switch:MX-NoLED MX6
+L tutorial-rescue:MX-NoLED-switch MX6
 U 1 1 5D11B01D
 P 10200 6400
@@
 $EndComp
 $Comp
-L switch:MX-NoLED MX7
+L tutorial-rescue:MX-NoLED-switch MX7
 U 1 1 5D11B373
 P 10700 6400
@@
 $EndComp
 $Comp
-L switch:MX-NoLED MX8
+L tutorial-rescue:MX-NoLED-switch MX8
 U 1 1 5D11B6C4
 P 10200 7400
@@
 $EndComp
 $Comp
-L switch:MX-NoLED MX9
+L tutorial-rescue:MX-NoLED-switch MX9
 U 1 1 5D11BEED
 P 10700 7400
